Commit message: update.

File: descriptions/urdf/dtw_robot/dtw_robot.urdf.xacro (robot description, xacro)
@@ -1,5 +1,5 @@
 <?xml version="1.0"?>
 <robot name="dtw_robot" xmlns:xacro="http://ros.org/wiki/xacro">
-    <!-- <xacro:arg name="robot_name" default="dtw_robot"/> -->
+    <xacro:arg name="robot_name" default="dtw_robot"/>
     <xacro:include filename="$(find descriptions)/urdf/dtw_robot/laser_macro.xacro"/>
     <xacro:include filename="$(find descriptions)/urdf/dtw_robot/imu_macro.xacro"/>
@@ -9,15 +9,12 @@
     <xacro:wheel_macro prefix="wheel_left" parent="base_link" xyz="0 0.1 0.05"/>
     <xacro:wheel_macro prefix="wheel_right" parent="base_link" xyz="0 -0.1 0.05"/>
-    <xacro:laser_macro prefix="front_laser" parent="base_link" xyz="0 0 0.13"/>
-    <!-- <xacro:imu_macro prefix="imu" parent="base_link" xyz="-0.05 0 0.10" robot_name="$(arg robot_name)"/> -->
-    <!-- <gazebo>
-        <plugin name="gazebo_ros_control" filename="libgazebo_ros_control.so">
-            <robotNamespace>$(arg robot_name)</robotNamespace>
-            <robotSimType>gazebo_ros_control/DefaultRobotHWSim</robotSimType>
-            <legacyModeNS>true</legacyModeNS>
-        </plugin>
-    </gazebo> -->
+    <!-- <xacro:laser_macro prefix="front_laser" parent="base_link" xyz="0 0 0.13"/> -->
+    <xacro:imu_macro prefix="imu" parent="base_link" xyz="-0.05 0 0.10" robot_name="$(arg robot_name)"/>
+    <xacro:include filename="$(find velodyne_description)/urdf/VLP-16.urdf.xacro"/>
+    <xacro:VLP-16 parent="base_link" name="velodyne" topic="/lidar_cloud2" organize_cloud="fasle" hz="10" samples="440" gpu="false">
+        <origin xyz="0 0 0.4" rpy="0 0 0" />
+    </xacro:VLP-16>
     <gazebo>
-        <plugin name="diff_drive" filename="libgazebo_ros_diff_drive.so">
+        <plugin name="diff_drive_plugin" filename="libgazebo_ros_diff_drive.so">
             <update_rate>30</update_rate>
             <!-- wheels -->
@@ -39,5 +36,5 @@
             <robot_base_frame>base_link</robot_base_frame>
         </plugin>
-        <plugin name="joint_state" filename="libgazebo_ros_joint_state_publisher.so">
+        <plugin name="joint_state_publisher_plugin" filename="libgazebo_ros_joint_state_publisher.so">
             <ros>
               <!-- <namespace>/br</namespace> -->

File: descriptions/urdf/dtw_robot/imu_macro.xacro (robot description, xacro)
@@ -9,22 +9,56 @@
     <link name="${prefix}_link"/>
     <gazebo reference="${prefix}_link">
-      <gravity>true</gravity>
-      <sensor name="imu_sensor" type="imu">
-        <always_on>true</always_on>
-        <update_rate>100</update_rate>
-        <visualize>true</visualize>
-        <topic>data</topic>
-        <plugin filename="libgazebo_ros_imu_sensor.so" name="imu_plugin">
-          <topicName>${prefix}/data</topicName>
-          <bodyName>${prefix}_link</bodyName>
-          <updateRateHZ>10.0</updateRateHZ>
-          <gaussianNoise>0.0</gaussianNoise>
-          <xyzOffset>0 0 0</xyzOffset>
-          <rpyOffset>0 0 0</rpyOffset>
-          <frameName>${robot_name}/${prefix}_link</frameName>
-        </plugin>
-        <pose>0 0 0 0 0 0</pose>
-      </sensor>
-    </gazebo>
+        <sensor name="imu_sensor" type="imu">
+          <always_on>true</always_on>
+            <update_rate>20</update_rate>
+            <imu>
+              <angular_velocity>
+                <x>
+                  <noise type="gaussian">
+                    <mean>0.0</mean>
+                    <stddev>2e-4</stddev>
+                  </noise>
+                </x>
+                <y>
+                  <noise type="gaussian">
+                    <mean>0.0</mean>
+                    <stddev>2e-4</stddev>
+                  </noise>
+                </y>
+                <z>
+                  <noise type="gaussian">
+                    <mean>0.0</mean>
+                    <stddev>2e-4</stddev>
+                  </noise>
+                </z>
+              </angular_velocity>
+              <linear_acceleration>
+                <x>
+                  <noise type="gaussian">
+                    <mean>0.0</mean>
+                    <stddev>1.7e-2</stddev>
+                  </noise>
+                </x>
+                <y>
+                  <noise type="gaussian">
+                    <mean>0.0</mean>
+                    <stddev>1.7e-2</stddev>
+                  </noise>
+                </y>
+                <z>
+                  <noise type="gaussian">
+                    <mean>0.0</mean>
+                    <stddev>1.7e-2</stddev>
+                  </noise>
+                </z>
+              </linear_acceleration>
+            </imu>
+            <!-- <plugin name="imu_plugin" filename="libgazebo_ros_imu_sensor.so">
+              <ros>
+                <remapping>~/out:=imu</remapping>
+              </ros>
+            </plugin> -->
+          </sensor>
+        </gazebo>
   </xacro:macro>
 </robot>
